Commit message: fix 03

File: lab5/ex03/my_robot/robot_description/urdf/robot.urdf.xacro (robot description, xacro)
@@ -43,5 +43,5 @@
       </material>
     </visual>
-        <collision>
+    <collision>
       <geometry>
         <box size="${base_length} ${base_width} ${base_height}"/>
@@ -86,5 +86,5 @@
   <xacro:wheel prefix="drivewhl_l" x_reflect="-1" y_reflect="1" />
   <xacro:wheel prefix="drivewhl_r" x_reflect="-1" y_reflect="-1" />
-    <!-- Caster Wheel -->
+  <!-- Caster Wheel -->
   <link name="front_caster">
     <visual>
@@ -96,5 +96,5 @@
       </material>
     </visual>
-        <collision>
+    <collision>
       <origin xyz="0 0 0" rpy="0 0 0"/>
       <geometry>
@@ -104,9 +104,8 @@
     <xacro:sphere_inertia m="0.5" r="${(wheel_radius+wheel_zoff-(base_height/2))}"/>
   </link>
-  <joint name="caster_joint" type="continuous">
+  <joint name="caster_joint" type="fixed">
     <parent link="base_link"/>
     <child link="front_caster"/>
     <origin xyz="${caster_xoff} 0.0 ${-(base_height/2)}" rpy="0 0 0"/>
-    <axis xyz="1 0 0"/>
   </joint>
 </robot>
