Commit message: fix ;)

File: lab6/ex05/my_robot/robot_description/urdf/depth.urdf.xacro (robot description, xacro)
@@ -5,5 +5,5 @@
         <parent link="base_link"/>
         <child link="depth_frame"/>
-        <origin xyz="0.1 0 0.25" rpy="0 0.2 0"/>
+        <origin xyz="0.6 0 0.55" rpy="0 0.2 0"/>
     </joint>
     <material name="aluminum">
